Commit message: fix urdf and usd for env vectorization

File: omniisaacgymenvs/models/franka_tekken/franka_tekken.urdf (robot description, URDF)
Before this commit: robot panda, 31 links, 30 joints
Links:
- link base_link_hithand: geometry collision mesh filename=./meshes/visual/tekken/palm-right.dae; visual mesh filename=./meshes/visual/tekken/palm-right.dae
